File: PCB/ButtonBoard/ButtonBoard.kicad_pcb (KiCad board)
At the start: 2 copper layers, 20 x 15 mm, 3 parts, among them J1 PAD, J2 PAD, SW1 SW_Push

Commit message: Generated gerbers
Other:
- board text added: "ButtonBoard v1"
Changed lines of the file:
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@@
   )
   (paper "A4")
+  (title_block
+    (title "ButtonBoard")
+    (date "2022-03-13")
+    (rev "v1")
+  )
   (layers
     (0 "F.Cu" signal)
@@
     (pad_to_mask_clearance 0.0508)
     (pcbplotparams
-      (layerselection 0x0000030_80000001)
+      (layerselection 0x00010f0_ffffffff)
       (disableapertmacros false)
-      (usegerberextensions false)
+      (usegerberextensions true)
       (usegerberattributes true)
       (usegerberadvancedattributes true)
@@
       (outputformat 1)
       (mirror false)
-      (drillshape 1)
+      (drillshape 0)
       (scaleselection 1)
-      (outputdirectory "")
+      (outputdirectory "plots/")
     )
   )
@@
   (gr_line (start 144.9 82.7) (end 144.9 99) (layer "F.Fab") (width 0.1))
   (gr_line (start 134 90.7) (end 156.4 90.7) (layer "F.Fab") (width 0.1))
-  (dimension (type aligned) (layer "F.Cu")
+  (gr_text "ButtonBoard v1" (at 144.9 90.7) (layer "B.SilkS")
+    (effects (font (size 1 1) (thickness 0.15)) (justify mirror))
+  )
+  (dimension (type aligned) (layer "Dwgs.User")
     (pts (xy 154.9 98.2) (xy 154.9 83.2))
     (height 6.8)
-    (gr_text "0.5906 in" (at 159.9 90.7 90) (layer "F.Cu")
+    (gr_text "15.0000 mm" (at 159.9 90.7 90) (layer "Dwgs.User")
       (effects (font (size 1.5 1.5) (thickness 0.3)))
     )
@@
     (style (thickness 0.2) (arrow_length 1.27) (text_position_mode 0) (extension_height 0.58642) (extension_offset 0.5) keep_text_aligned)
   )
-  (dimension (type aligned) (layer "F.Cu")
+  (dimension (type aligned) (layer "Dwgs.User")
     (pts (xy 134.9 98.2) (xy 154.9 98.2))
     (height 4.6)
-    (gr_text "0.7874 in" (at 144.9 101) (layer "F.Cu")
+    (gr_text "20.0000 mm" (at 144.9 101) (layer "Dwgs.User")
       (effects (font (size 1.5 1.5) (thickness 0.3)))
     )
